Commit message: feat: Motorlar döndü (DM860H), STM32-Pi doğrudan UART, açılış bekçisi ve kararlılık düzeltmeleri
Motor sürücü (DM860H + 86HS156 step motor):
- STM32 yazılımı 1.3.1: motor pinleri open-drain (DM860H 5 V ortak anot
  girişleri için), STEP kutbu ters (dururken opto sönük), EN aktif-yüksek,
  teker başına yön tersleme (sağ teker ters - tezgâhta doğrulandı).
- Uçtan uca doğrulandı: telefon/cmd_vel -> Pi -> STM32 -> DM860H -> motor.

STM32 <-> Pi haberleşmesi:
- Nucleo'nun ST-LINK seri köprüsü 5V kısa devresinde bozuldu; haberleşme
  USART3'e (PC10/PC11) taşındı, Pi tarafında /dev/ttyAMA0 (udev kuralı
  güncellendi). PI_LINK_USART3=0 ile eski yola dönülebilir.
- UART hata (overrun/framing) sonrası alım artık kendiliğinden yeniden
  başlıyor; eskiden tek bir parazit STM32'yi kalıcı "sağır" bırakıyordu.

Robot yazılımı:
- Nav2 açılış bekçisi: açılışta lifecycle yöneticileri kilitlenirse Nav2
  75 sn sonra otomatik yeniden başlatılıyor (en fazla 3 deneme).
- Sonar çerçeveleri URDF'ye eklendi (range_layer artık sonarları kullanıyor).
- Batarya takılı değilken (<5 V) "batarya düşük" diye devriye durdurulmuyor.
- Servis: SIGINT ile temiz kapanma, 20 sn zaman aşımı ve Fast DDS kalıntı
  temizliği (bozuk paylaşımlı bellek yüzünden robot hiç açılmıyordu).
- Kafa ekranı: animasyonlar tek bir 20 kare/sn saatine bağlandı,
  Chromium CPU yükü %116 -> %75.

Diğer: Flutter testi güncellendi, README'de Pi 4 GB ve IMU durumu düzeltildi.

Co-Authored-By: Claude Opus 5.5 <noreply@anthropic.com>

File: cryvex_hw_ws/src/cryvex_bringup/urdf/cryvex_real.urdf.xacro (robot description, xacro)
@@ -67,4 +67,31 @@
     <origin xyz="0 0 ${lidar_height}" rpy="0 0 0"/>
   </joint>
+  <!-- ============ 4x HC-SR04 (STM32 -> stm32_bridge -> /ultrasonic/*) ============
+       stm32_bridge her Range mesajini frame_id = sonar_{fl,fr,rl,rr}_link ile
+       yayinlar; Nav2'nin range_layer'i (nav2_params.yaml) sonari costmap'e
+       islemek icin bu cercevelere TF ister. 2026-10-01'e kadar bu linkler
+       YOKTU -> range_layer her 2.5 sn "frame does not exist" uyarip sonarlari
+       hic kullanmiyordu.
+       Yerlesim sim'de (cryvex.urdf.xacro) test edilen duzenin aynisi: ondeki
+       iki sensor +-17 derece iceri bakar, +-20 derecelik huzmeleri TAM ONDE ust
+       uste biner (kor nokta yok); arkada da ayni.
+       OLCULER YER TUTUCU: govde kurulunca sensorlerin gercek konumunu olcup
+       asagidaki 4 property'yi guncelleyin (TF yapisi degismez). -->
+  <xacro:property name="sonar_x" value="0.30"/>     <!-- merkezden one/arkaya (m) -->
+  <xacro:property name="sonar_y" value="0.13"/>     <!-- merkezden sola/saga (m) -->
+  <xacro:property name="sonar_z" value="0.10"/>     <!-- zeminden yukseklik (m) -->
+  <xacro:property name="sonar_yaw" value="0.30"/>   <!-- ice donukluk (rad, ~17 derece) -->
+  <xacro:macro name="sonar" params="name x y yaw">
+    <link name="sonar_${name}_link"/>
+    <joint name="base_link_to_sonar_${name}" type="fixed">
+      <parent link="base_link"/>
+      <child link="sonar_${name}_link"/>
+      <origin xyz="${x} ${y} ${sonar_z}" rpy="0 0 ${yaw}"/>
+    </joint>
+  </xacro:macro>
+  <xacro:sonar name="fl" x="${sonar_x}"  y="${sonar_y}"  yaw="${sonar_yaw}"/>
+  <xacro:sonar name="fr" x="${sonar_x}"  y="${-sonar_y}" yaw="${-sonar_yaw}"/>
+  <xacro:sonar name="rl" x="${-sonar_x}" y="${sonar_y}"  yaw="${pi - sonar_yaw}"/>
+  <xacro:sonar name="rr" x="${-sonar_x}" y="${-sonar_y}" yaw="${-pi + sonar_yaw}"/>
   <!-- MPU6050 - stm32_bridge.py sadece Z ekseni acisal hizini yayinliyor,
        konum onemsiz; kart DUZ (Z yukari) monte edilmezse buraya rpy eklenmeli. -->

Commit message: fix: Robotun kendi etrafında dönmesi ve haritanın bozulması - teker yönü, iz genişliği ve LiDAR konumu ölçülerek düzeltildi
LiDAR'ı referans alan ölçüm testiyle (90° dönüş + 50 cm ileri, tarama
eşleştirme/ICP) üç ayrı hata bulundu:

- Teker yönü: tezgâhta ters çevrilen sağ teker, tabana takılınca yanlış
  çıktı; "ileri" komutunda robot yerinde dönüyordu (STM32 1.3.3).
- İz genişliği: yer tutucu 400 mm, ölçülen 540 mm; odometri dönüşleri
  %40 fazla sayıyordu (STM32 1.3.4 + stm32_bridge). Teker çapı 150 mm doğru.
- LiDAR konumu: tabanın en yüksek noktasına kaçık ve dönük takılmış;
  URDF'de x=0.104 y=-0.124 yaw=-128°. Eski değerle 50 cm ilerleyince
  duvarlar haritada ~48 cm kayıyordu, yenisiyle ~5 cm.

Sonuç: dönüş %97, ileri %96 uyum. slam_toolbox'ın motorsuz dönem için
konan "her taramayı işle" ayarları kaldırıldı (0.2 m / 0.2 rad).

Co-Authored-By: Claude Opus 5.5 <noreply@anthropic.com>

File: cryvex_hw_ws/src/cryvex_bringup/urdf/cryvex_real.urdf.xacro (robot description, xacro)
@@ -25,4 +25,16 @@
   <xacro:property name="base_height" value="0.12"/>
   <xacro:property name="lidar_height" value="0.22"/>  <!-- malzeme listesi rev.4, bolum 5: "yerden ~20-30 cm" -->
+  <!-- 2026-10-02: LiDAR tabanin en yuksek noktasina, merkezden kacik ve donuk
+       takildi. Konum/aci LiDAR'in kendisiyle OLCULDU (90 derece donus + 50 cm ileri
+       testi, tarama eslestirme/ICP): teker ekseni ortasina gore ~10 cm onde,
+       ~12 cm sagda, LiDAR'in 0 derece yonu robotun onune gore -128 derece.
+       Eski degerle (merkez, 0 derece) robot 50 cm ilerleyince duvarlar haritada
+       ~48 cm kayiyordu; bu degerlerle ~5 cm. "On" = robotun +x yonu (STM32
+       *_WHEEL_DIR_INVERT ayarina gore ileri gittigi taraf). Ekran tarafi on
+       olacaksa: iki teker terslemesini de cevirin, lidar_x/lidar_y'nin isaretini
+       degistirin ve lidar_yaw'a 180 derece ekleyin (-128 -> +52). -->
+  <xacro:property name="lidar_x" value="0.104"/>
+  <xacro:property name="lidar_y" value="-0.124"/>
+  <xacro:property name="lidar_yaw" value="${radians(-128)}"/>
   <material name="cryvex_dark">
     <color rgba="0.08 0.08 0.10 1.0"/>
@@ -65,5 +77,5 @@
     <parent link="base_link"/>
     <child link="lidar_link"/>
-    <origin xyz="0 0 ${lidar_height}" rpy="0 0 0"/>
+    <origin xyz="${lidar_x} ${lidar_y} ${lidar_height}" rpy="0 0 ${lidar_yaw}"/>
   </joint>
   <!-- ============ 4x HC-SR04 (STM32 -> stm32_bridge -> /ultrasonic/*) ============

Commit message: fix: Nav2 robot yarıçapı 0.35 -> 0.30 m (gövde 52 cm daire, tekerler 54 cm aralıklı)
Co-Authored-By: Claude Opus 5.5 <noreply@anthropic.com>

File: cryvex_hw_ws/src/cryvex_bringup/urdf/cryvex_real.urdf.xacro (robot description, xacro)
@@ -22,5 +22,5 @@
 -->
 <robot name="cryvex_real" xmlns:xacro="http://www.ros.org/wiki/xacro">
-  <xacro:property name="footprint_radius" value="0.35"/>
+  <xacro:property name="footprint_radius" value="0.30"/>  <!-- 2026-10-02: govde 52 cm daire + tasan tekerler -->
   <xacro:property name="base_height" value="0.12"/>
   <xacro:property name="lidar_height" value="0.22"/>  <!-- malzeme listesi rev.4, bolum 5: "yerden ~20-30 cm" -->

Commit message: fix: SLAM tarama eşleştirici odometriye yakın kalıyor; LiDAR açısı -123 derece
slam_toolbox varsayılanları odometriyi neredeyse hiç cezalandırmıyordu,
kalabalık ortamda yanlış eşleşmeyle konum 0.05<->0.87 m / 16 derece zıplıyor
ve harita katlanıyordu. Teker + LiDAR ICP %3 içinde uyumlu olduğu için
eşleştirme penceresi daraltıldı, sapma cezası artırıldı, döngü kapatma
daha seçici, menzil 8 m. Düz gidiş testinden LiDAR yaw -128 -> -123,
konum 0.103/-0.131.

Co-Authored-By: Claude Opus 5.5 <noreply@anthropic.com>

File: cryvex_hw_ws/src/cryvex_bringup/urdf/cryvex_real.urdf.xacro (robot description, xacro)
@@ -33,8 +33,12 @@
        *_WHEEL_DIR_INVERT ayarina gore ileri gittigi taraf). Ekran tarafi on
        olacaksa: iki teker terslemesini de cevirin, lidar_x/lidar_y'nin isaretini
-       degistirin ve lidar_yaw'a 180 derece ekleyin (-128 -> +52). -->
-  <xacro:property name="lidar_x" value="0.104"/>
-  <xacro:property name="lidar_y" value="-0.124"/>
-  <xacro:property name="lidar_yaw" value="${radians(-128)}"/>
+       degistirin ve lidar_yaw'a 180 derece ekleyin (-123 -> +57).
+       2026-10-02 (2. olcum): temiz koridorda 0.39 m duz ileri/geri + yerinde
+       +-90 derece testi -> yaw -128 degil -123 (5 derece fark 1 m'de ~9 cm yana
+       kayma demek), konum 0.103/-0.131. Bu degerlerle teker odometrisiyle
+       tasinan iki tarama dunyada ust uste biniyor. -->
+  <xacro:property name="lidar_x" value="0.103"/>
+  <xacro:property name="lidar_y" value="-0.131"/>
+  <xacro:property name="lidar_yaw" value="${radians(-123)}"/>
   <material name="cryvex_dark">
     <color rgba="0.08 0.08 0.10 1.0"/>

Commit message: merge: 5-8 Ekim robot çalışması ana depoya birleştirildi (kamera + YOLO, LiDAR odometrisi, güvenlik kapısı, HOME-Masa görevi)
Kaynak: yigithan1318yts/cryvex-maskot-robot (8 Ekim anlık kopyası, taban 80c9808).
Kod dosyalarında satır çakışması yok - taban sonrası bizde yalnızca belge değişti.

Alınanlar:
- cryvex_bringup: rf2o ile EKF dönüşü, stm32_bridge YON_DUZELTME + sıçrama
  filtresi + pencereli hız, SLAM penceresi ±25 cm/±20°, otonom.launch.py +
  nav2_otonom.yaml + davranış ağaçları, /otonom sayfası ve /api/otonom,
  canlı harita önbelleği, tek tur devriye, LiDAR yeni montaj (36 cm, -90°)
- src/rf2o_laser_odometry, src/frontier_exploration_ros2 (lisanslarıyla)
- cryvex_araclar/ (Pi: ~/cryvex_araclar), cryvex_veri/ (Pi: ~/cryvex_veri)
- docs: GUNLUK.md, mimari_v1.md, robot_alisveris_listesi.md, resimler/

Birleştirmede düzeltilenler:
- algılama yalnızca ~/cryvex_ai ve algilama.py varsa başlatılıyor
- URDF açıklaması yeni LiDAR montajına göre güncellendi
- README'den IP kaldırıldı, 'STM32 kaynağı yok' düzeltildi
- siparişler, son konum, kayıtlar, eski haritalar, .pt ve MobileNet git dışı
- gercek_robot.md ve README 8 Ekim durumuna göre güncellendi

Co-Authored-By: Claude Opus 5.5 <noreply@anthropic.com>

File: cryvex_hw_ws/src/cryvex_bringup/urdf/cryvex_real.urdf.xacro (robot description, xacro)
@@ -22,23 +22,19 @@
 -->
 <robot name="cryvex_real" xmlns:xacro="http://www.ros.org/wiki/xacro">
-  <xacro:property name="footprint_radius" value="0.30"/>  <!-- 2026-10-02: govde 52 cm daire + tasan tekerler -->
+  <xacro:property name="footprint_radius" value="0.30"/>  <!-- 2026-10-05: tekerden tekere 59 cm olculdu (R 0.295), 0.30 korundu -->
   <xacro:property name="base_height" value="0.12"/>
-  <xacro:property name="lidar_height" value="0.22"/>  <!-- malzeme listesi rev.4, bolum 5: "yerden ~20-30 cm" -->
-  <!-- 2026-10-02: LiDAR tabanin en yuksek noktasina, merkezden kacik ve donuk
-       takildi. Konum/aci LiDAR'in kendisiyle OLCULDU (90 derece donus + 50 cm ileri
-       testi, tarama eslestirme/ICP): teker ekseni ortasina gore ~10 cm onde,
-       ~12 cm sagda, LiDAR'in 0 derece yonu robotun onune gore -128 derece.
-       Eski degerle (merkez, 0 derece) robot 50 cm ilerleyince duvarlar haritada
-       ~48 cm kayiyordu; bu degerlerle ~5 cm. "On" = robotun +x yonu (STM32
-       *_WHEEL_DIR_INVERT ayarina gore ileri gittigi taraf). Ekran tarafi on
-       olacaksa: iki teker terslemesini de cevirin, lidar_x/lidar_y'nin isaretini
-       degistirin ve lidar_yaw'a 180 derece ekleyin (-123 -> +57).
-       2026-10-02 (2. olcum): temiz koridorda 0.39 m duz ileri/geri + yerinde
-       +-90 derece testi -> yaw -128 degil -123 (5 derece fark 1 m'de ~9 cm yana
-       kayma demek), konum 0.103/-0.131. Bu degerlerle teker odometrisiyle
-       tasinan iki tarama dunyada ust uste biniyor. -->
-  <xacro:property name="lidar_x" value="0.103"/>
-  <xacro:property name="lidar_y" value="-0.131"/>
-  <xacro:property name="lidar_yaw" value="${radians(-123)}"/>
+  <xacro:property name="lidar_height" value="0.36"/>  <!-- 2026-10-05: kamera eklenirken LiDAR yukseltildi, yerden 36 cm -->
+  <!-- LiDAR konumu/acisi - GECERLI DEGERLER (2026-10-05, robotta calisan kurulum):
+       LiDAR kamera taretiyle birlikte YENIDEN TAKILDI; ayni zamanda robotun
+       "on"u ters cevrildi (stm32_bridge.py YON_DUZELTME: ileri komutunun isareti
+       ve sol/sag teker sayaclari Pi tarafinda cevriliyor, STM32 yazilimi ayni).
+       Bu yuzden 2026-10-02'deki ICP olcumleri (x 0.103, y -0.131, yaw -123)
+       artik GECERSIZ - eski govdeye ve eski "on"a aitti.
+       Yeniden olcmek icin: docs/gercek_robot.md "LiDAR'i cetvel olarak kullanmak".
+       Not: LiDAR duzlemi 36 cm'de; bunun altindaki masa ayagi tabani, kablo,
+       palet alti gorulmez (bkz. docs/GUNLUK.md, ToF sensorleri planli). -->
+  <xacro:property name="lidar_x" value="0.125"/>
+  <xacro:property name="lidar_y" value="-0.045"/>
+  <xacro:property name="lidar_yaw" value="${radians(-90)}"/>
   <material name="cryvex_dark">
     <color rgba="0.08 0.08 0.10 1.0"/>

Commit message: feat: Sekizgen gövde - 6 ultrasonik sensör 60 derecede bir, dışarı bakan yerleşim
URDF: sonar konumu açı + sekizgen iç yarıçapından (sekizgen_a, şimdilik 0.26 m)
hesaplanır: fc 0, fl +60, rl +120, rc 180, rr -120, fr -60. ±60/±120'dekiler
45/135'lik kenarda, merkeze sekizgen_a/cos15 uzaklıkta, kenara 15° eğik.
patrol SONAR_YAW aynı açılara güncellendi. Belge: montaj şeması ve kör bölgeler.

Co-Authored-By: Claude Opus 5.5 <noreply@anthropic.com>

File: cryvex_hw_ws/src/cryvex_bringup/urdf/cryvex_real.urdf.xacro (robot description, xacro)
@@ -79,34 +79,35 @@
     <origin xyz="${lidar_x} ${lidar_y} ${lidar_height}" rpy="0 0 ${lidar_yaw}"/>
   </joint>
-  <!-- ============ 6x HC-SR04 (STM32 -> stm32_bridge -> /ultrasonic/*) ============
-       stm32_bridge her Range mesajini frame_id = sonar_{fl,fr,rl,rr}_link ile
-       yayinlar; Nav2'nin range_layer'i (nav2_params.yaml) sonari costmap'e
-       islemek icin bu cercevelere TF ister. 2026-10-01'e kadar bu linkler
-       YOKTU -> range_layer her 2.5 sn "frame does not exist" uyarip sonarlari
-       hic kullanmiyordu.
-       Yerlesim sim'de (cryvex.urdf.xacro) test edilen duzenin aynisi: ondeki
-       iki sensor +-17 derece iceri bakar, +-20 derecelik huzmeleri TAM ONDE ust
-       uste biner (kor nokta yok); arkada da ayni.
-       OLCULER YER TUTUCU: govde kurulunca sensorlerin gercek konumunu olcup
-       asagidaki 4 property'yi guncelleyin (TF yapisi degismez). -->
-  <xacro:property name="sonar_x" value="0.30"/>     <!-- merkezden one/arkaya (m) -->
-  <xacro:property name="sonar_y" value="0.13"/>     <!-- merkezden sola/saga (m) -->
-  <xacro:property name="sonar_z" value="0.10"/>     <!-- zeminden yukseklik (m) -->
-  <xacro:property name="sonar_yaw" value="0.30"/>   <!-- ice donukluk (rad, ~17 derece) -->
-  <xacro:macro name="sonar" params="name x y yaw">
+  <!-- ============ 6x HC-SR04 (STM32 1.4.0 -> stm32_bridge -> /ultrasonic/*) ============
+       stm32_bridge her Range mesajini frame_id = sonar_<ad>_link ile yayinlar;
+       Nav2'nin range katmani bu cercevelere TF ister.
+       2026-10-23 YERLESIM: govde SEKIZGEN, 6 sensor cevrede ESIT ARALIKLA (60
+       derecede bir), hepsi merkezden DISARI bakar ("on" = +x = kamera tarafi):
+                       fc 0
+             fl +60          fr -60
+             rl +120         rr -120
+                      rc 180
+       Sekizgenin kenar normalleri 0/45/90/135... derecede. 0 ve 180'deki sensor
+       kenar ortasinda (merkeze uzaklik = sekizgen_a); +-60 ve +-120'dekiler
+       45/135'lik kenarda, kose tarafina 15 derece kaymis noktada:
+       uzaklik = sekizgen_a / cos(15 derece), sensor kenara gore 15 derece
+       egik (dis bakan) takilir.
+       OLCULER YER TUTUCU: govde bitince sekizgen_a ve sonar_z'yi olcun. -->
+  <xacro:property name="sekizgen_a" value="0.26"/>   <!-- merkezden kenar ortasina (m); karsilikli kenarlar arasi / 2 -->
+  <xacro:property name="sonar_z" value="0.12"/>      <!-- zeminden yukseklik (m) -->
+  <xacro:macro name="sonar" params="name aci r">
     <link name="sonar_${name}_link"/>
     <joint name="base_link_to_sonar_${name}" type="fixed">
       <parent link="base_link"/>
       <child link="sonar_${name}_link"/>
-      <origin xyz="${x} ${y} ${sonar_z}" rpy="0 0 ${yaw}"/>
+      <origin xyz="${r*cos(radians(aci))} ${r*sin(radians(aci))} ${sonar_z}" rpy="0 0 ${radians(aci)}"/>
     </joint>
   </xacro:macro>
-  <xacro:sonar name="fl" x="${sonar_x}"  y="${sonar_y}"  yaw="${sonar_yaw}"/>
-  <xacro:sonar name="fr" x="${sonar_x}"  y="${-sonar_y}" yaw="${-sonar_yaw}"/>
-  <xacro:sonar name="rl" x="${-sonar_x}" y="${sonar_y}"  yaw="${pi - sonar_yaw}"/>
-  <xacro:sonar name="rr" x="${-sonar_x}" y="${-sonar_y}" yaw="${-pi + sonar_yaw}"/>
-  <!-- 2026-10-23: 6 sensor (STM32 1.4.0) - on orta ve arka orta -->
-  <xacro:sonar name="fc" x="${sonar_x}"  y="0"            yaw="0"/>
-  <xacro:sonar name="rc" x="${-sonar_x}" y="0"            yaw="${pi}"/>
+  <xacro:sonar name="fc" aci="0"    r="${sekizgen_a}"/>
+  <xacro:sonar name="fl" aci="60"   r="${sekizgen_a/cos(radians(15))}"/>
+  <xacro:sonar name="rl" aci="120"  r="${sekizgen_a/cos(radians(15))}"/>
+  <xacro:sonar name="rc" aci="180"  r="${sekizgen_a}"/>
+  <xacro:sonar name="rr" aci="-120" r="${sekizgen_a/cos(radians(15))}"/>
+  <xacro:sonar name="fr" aci="-60"  r="${sekizgen_a/cos(radians(15))}"/>
   <!-- MPU6050 - stm32_bridge.py sadece Z ekseni acisal hizini yayinliyor,
        konum onemsiz; kart DUZ (Z yukari) monte edilmezse buraya rpy eklenmeli. -->

Commit message: fix: Robotun gerçek şekli Nav2'ye verildi (ön uç 45 cm, daire 30 sanıyordu); LiDAR 30 cm, iç ölçümler filtrelendi
Kullanıcı ölçüleri (2026-10-23): sekizgen gövde, merkezden kenara 30 cm (kenar
23 cm), LiDAR gövdenin TAM merkezinde yerden 30 cm, 0 derecesi robotun sağına
bakıyor (yanlış yapıştırılmış; yaw -90 zaten doğru), etrafında ~25 cm'de 4 destek.
Dönüş kaydından LiDAR dönme merkezinin (teker ekseni) 13.5 cm önünde -> teker
ekseni gövde merkezinin gerisinde; ön uç dönme merkezinden 45 cm ileride, arka
18 cm. Nav2 robotu dönme merkezi etrafında 0.30'luk daire sanıyordu (önü 15 cm
kısa) - masa ayağı çarpmasıyla uyumlu.
- nav2_params / nav2_otonom: robot_radius -> footprint (sekizgen + tekerler +
  2 cm, 10 köşe); inflation_radius 0.50/0.55 -> 0.65 (en uzak nokta 0.49 m).
  collision_monitor ayak izini /local_costmap/published_footprint'ten alır.
- URDF: lidar_height 0.30, lidar_x 0.135; sonarlar gövde merkezine göre
  (sekizgen_a 0.30).
- YDLIDAR range_min 0.03 -> 0.33: 33 cm içinde yalnız robotun kendisi var
  (destekler, kablolar).
ROBOTTA HENÜZ DOĞRULANMADI.

Co-Authored-By: Claude Opus 5.5 <noreply@anthropic.com>

File: cryvex_hw_ws/src/cryvex_bringup/urdf/cryvex_real.urdf.xacro (robot description, xacro)
@@ -24,5 +24,5 @@
   <xacro:property name="footprint_radius" value="0.30"/>  <!-- 2026-10-05: tekerden tekere 59 cm olculdu (R 0.295), 0.30 korundu -->
   <xacro:property name="base_height" value="0.12"/>
-  <xacro:property name="lidar_height" value="0.36"/>  <!-- 2026-10-05: kamera eklenirken LiDAR yukseltildi, yerden 36 cm -->
+  <xacro:property name="lidar_height" value="0.30"/>  <!-- 2026-10-23: kullanici olctu - yerden 30 cm, govdenin TAM merkezinde -->
   <!-- LiDAR konumu/acisi - GECERLI DEGERLER (2026-10-05, robotta calisan kurulum):
        LiDAR kamera taretiyle birlikte YENIDEN TAKILDI; ayni zamanda robotun
@@ -34,5 +34,11 @@
        Not: LiDAR duzlemi 36 cm'de; bunun altindaki masa ayagi tabani, kablo,
        palet alti gorulmez (bkz. docs/GUNLUK.md, ToF sensorleri planli). -->
-  <xacro:property name="lidar_x" value="0.125"/>
+  <!-- 2026-10-23: LiDAR sekizgen govdenin TAM MERKEZINDE (kullanici). Robot teker ekseni
+       ortasi (base_link) etrafinda doner; donus kaydindan (LiDAR ICP, 43 olcum, 0.8 cm artik)
+       LiDAR'in bu noktaya gore yeri x +0.135 y -0.045 bulundu -> teker ekseni govde
+       merkezinin ~13.5 cm GERISINDE. LiDAR'in 0 derecesi robotun tam SAGINA bakiyor
+       (yanlis yonde yapistirildi, kullanici dogruladi) -> yaw -90. Nav2 ayak izi bu
+       geometriden hesaplandi (nav2_params.yaml 'footprint'). -->
+  <xacro:property name="lidar_x" value="0.135"/>
   <xacro:property name="lidar_y" value="-0.045"/>
   <xacro:property name="lidar_yaw" value="${radians(-90)}"/>
@@ -88,5 +94,5 @@
              rl +120         rr -120
                       rc 180
-       Sekizgenin kenar normalleri 0/45/90/135... derecede. 0 ve 180'deki sensor
+       Sekizgenin merkezi LiDAR'da (teker ekseninin ~13.5 cm onunde). Kenar normalleri 0/45/90/135... derecede. 0 ve 180'deki sensor
        kenar ortasinda (merkeze uzaklik = sekizgen_a); +-60 ve +-120'dekiler
        45/135'lik kenarda, kose tarafina 15 derece kaymis noktada:
@@ -94,5 +100,8 @@
        egik (dis bakan) takilir.
        OLCULER YER TUTUCU: govde bitince sekizgen_a ve sonar_z'yi olcun. -->
-  <xacro:property name="sekizgen_a" value="0.26"/>   <!-- merkezden kenar ortasina (m); karsilikli kenarlar arasi / 2 -->
+  <xacro:property name="sekizgen_a" value="0.30"/>   <!-- 2026-10-23 olculdu: merkezden kenar ortasina 30 cm (kenar 23 cm) -->
+  <!-- Sekizgenin merkezi = LiDAR (yukarida); sensorler bu merkeze gore yerlesir. -->
+  <xacro:property name="govde_x" value="${lidar_x}"/>
+  <xacro:property name="govde_y" value="${lidar_y}"/>
   <xacro:property name="sonar_z" value="0.12"/>      <!-- zeminden yukseklik (m) -->
   <xacro:macro name="sonar" params="name aci r">
@@ -101,5 +110,5 @@
       <parent link="base_link"/>
       <child link="sonar_${name}_link"/>
-      <origin xyz="${r*cos(radians(aci))} ${r*sin(radians(aci))} ${sonar_z}" rpy="0 0 ${radians(aci)}"/>
+      <origin xyz="${govde_x + r*cos(radians(aci))} ${govde_y + r*sin(radians(aci))} ${sonar_z}" rpy="0 0 ${radians(aci)}"/>
     </joint>
   </xacro:macro>
